File: Bike Safety.kicad_sch (KiCad schematic)
At the start: 15 parts, among them U1 WeMos_D1_mini, U2 HC-SR04, U3 SW-420

Commit message: Add files via upload
Parts:
- added R7: 10k, symbol Device:R
- added SW1: SW_Push, symbol Switch:SW_Push
Connections:
- net +5V: now also SW1.2
- net GND: now also R7.2
- net at U1.7 (CS/D8): now also R7.1, SW1.1
Changed lines of the file:
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@@
 (kicad_sch (version 20230121) (generator eeschema)
   (paper "A4")
+  (junction (at 160.02 133.35) (diameter 0) (color 0 0 0 0)
+  )
   (junction (at 176.53 77.47) (diameter 0) (color 0 0 0 0)
   )
@@
     (stroke (width 0) (type default))
   )
+  (wire (pts (xy 160.02 134.62) (xy 160.02 133.35))
+    (stroke (width 0) (type default))
+  )
   (wire (pts (xy 90.17 64.77) (xy 93.98 64.77))
     (stroke (width 0) (type default))
@@
     (stroke (width 0) (type default))
   )
+  (wire (pts (xy 149.86 133.35) (xy 160.02 133.35))
+    (stroke (width 0) (type default))
+  )
   (wire (pts (xy 149.86 95.25) (xy 190.5 95.25))
+    (stroke (width 0) (type default))
+  )
+  (wire (pts (xy 149.86 102.87) (xy 149.86 133.35))
     (stroke (width 0) (type default))
   )
@@
     (pin "1")
     (instances
-      (project "Bike Safety"
+      (project "Bike Safety-2"
         (path "/1925ab50-b129-485f-aa70-9d722d7d68aa"
           (reference "#PWR05") (unit 1)
@@
     (pin "1")
     (instances
-      (project "Bike Safety"
+      (project "Bike Safety-2"
         (path "/1925ab50-b129-485f-aa70-9d722d7d68aa"
           (reference "#PWR01") (unit 1)
@@
     (pin "2")
     (instances
-      (project "Bike Safety"
+      (project "Bike Safety-2"
         (path "/1925ab50-b129-485f-aa70-9d722d7d68aa"
           (reference "D3") (unit 1)
@@
     )
   )
+  (symbol (lib_id "power:GND") (at 160.02 142.24 0) (unit 1)
+    (in_bom yes) (on_board yes) (dnp no) (fields_autoplaced)
+    (property "Reference" "#PWR014" (at 160.02 148.59 0)
+      (effects (font (size 1.27 1.27)) hide)
+    )
+    (property "Value" "GND" (at 160.02 147.32 0)
+      (effects (font (size 1.27 1.27)))
+    )
+    (property "Footprint" "" (at 160.02 142.24 0)
+      (effects (font (size 1.27 1.27)) hide)
+    )
+    (property "Datasheet" "" (at 160.02 142.24 0)
+      (effects (font (size 1.27 1.27)) hide)
+    )
+    (pin "1")
+    (instances
+      (project "Bike Safety-2"
+        (path "/1925ab50-b129-485f-aa70-9d722d7d68aa"
+          (reference "#PWR014") (unit 1)
+        )
+      )
+    )
+  )
   (symbol (lib_id "Device:R") (at 162.56 113.03 270) (unit 1)
     (in_bom yes) (on_board yes) (dnp no) (fields_autoplaced)
@@
     (pin "2")
     (instances
-      (project "Bike Safety"
+      (project "Bike Safety-2"
         (path "/1925ab50-b129-485f-aa70-9d722d7d68aa"
           (reference "R1") (unit 1)
@@
     (pin "2")
     (instances
-      (project "Bike Safety"
+      (project "Bike Safety-2"
         (path "/1925ab50-b129-485f-aa70-9d722d7d68aa"
           (reference "R4") (unit 1)
@@
     (pin "2")
     (instances
-      (project "Bike Safety"
+      (project "Bike Safety-2"
         (path "/1925ab50-b129-485f-aa70-9d722d7d68aa"
           (reference "R6") (unit 1)
@@
     (pin "2")
     (instances
-      (project "Bike Safety"
+      (project "Bike Safety-2"
         (path "/1925ab50-b129-485f-aa70-9d722d7d68aa"
           (reference "R3") (unit 1)
@@
     (pin "1")
     (instances
-      (project "Bike Safety"
+      (project "Bike Safety-2"
         (path "/1925ab50-b129-485f-aa70-9d722d7d68aa"
           (reference "#PWR08") (unit 1)
@@
     (pin "1")
     (instances
-      (project "Bike Safety"
+      (project "Bike Safety-2"
         (path "/1925ab50-b129-485f-aa70-9d722d7d68aa"
           (reference "#PWR02") (unit 1)
@@
     (pin "1")
     (instances
-      (project "Bike Safety"
+      (project "Bike Safety-2"
         (path "/1925ab50-b129-485f-aa70-9d722d7d68aa"
           (reference "#PWR013") (unit 1)
@@
     (pin "1")
     (instances
-      (project "Bike Safety"
+      (project "Bike Safety-2"
         (path "/1925ab50-b129-485f-aa70-9d722d7d68aa"
           (reference "#PWR07") (unit 1)
@@
     (pin "2")
     (instances
-      (project "Bike Safety"
+      (project "Bike Safety-2"
         (path "/1925ab50-b129-485f-aa70-9d722d7d68aa"
           (reference "R5") (unit 1)
@@
     (pin "2")
     (instances
-      (project "Bike Safety"
+      (project "Bike Safety-2"
         (path "/1925ab50-b129-485f-aa70-9d722d7d68aa"
           (reference "D2") (unit 1)
@@
       (effects (font (size 1.27 1.27)) hide)
     )
+    (pin "1")
     (pin "1")
     (pin "10")
@@
     (pin "8")
     (pin "9")
-    (pin "1")
-    (instances
-      (project "Bike Safety"
+    (instances
+      (project "Bike Safety-2"
         (path "/1925ab50-b129-485f-aa70-9d722d7d68aa"
           (reference "U1") (unit 1)
@@
     (pin "2")
     (instances
-      (project "Bike Safety"
+      (project "Bike Safety-2"
         (path "/1925ab50-b129-485f-aa70-9d722d7d68aa"
           (reference "D1") (unit 1)
@@
     (pin "1")
     (instances
-      (project "Bike Safety"
+      (project "Bike Safety-2"
         (path "/1925ab50-b129-485f-aa70-9d722d7d68aa"
           (reference "#PWR010") (unit 1)
@@
     (pin "2")
     (instances
-      (project "Bike Safety"
+      (project "Bike Safety-2"
         (path "/1925ab50-b129-485f-aa70-9d722d7d68aa"
           (reference "BT1") (unit 1)
@@
     )
   )
+  (symbol (lib_id "power:+5V") (at 160.02 123.19 0) (unit 1)
+    (in_bom yes) (on_board yes) (dnp no) (fields_autoplaced)
+    (property "Reference" "#PWR015" (at 160.02 127 0)
+      (effects (font (size 1.27 1.27)) hide)
+    )
+    (property "Value" "+5V" (at 160.02 118.11 0)
+      (effects (font (size 1.27 1.27)))
+    )
+    (property "Footprint" "" (at 160.02 123.19 0)
+      (effects (font (size 1.27 1.27)) hide)
+    )
+    (property "Datasheet" "" (at 160.02 123.19 0)
+      (effects (font (size 1.27 1.27)) hide)
+    )
+    (pin "1")
+    (instances
+      (project "Bike Safety-2"
+        (path "/1925ab50-b129-485f-aa70-9d722d7d68aa"
+          (reference "#PWR015") (unit 1)
+        )
+      )
+    )
+  )
   (symbol (lib_id "power:GND") (at 90.17 77.47 0) (unit 1)
     (in_bom yes) (on_board yes) (dnp no) (fields_autoplaced)
@@
     (pin "1")
     (instances
-      (project "Bike Safety"
+      (project "Bike Safety-2"
         (path "/1925ab50-b129-485f-aa70-9d722d7d68aa"
           (reference "#PWR03") (unit 1)
@@
     (pin "1")
     (instances
-      (project "Bike Safety"
+      (project "Bike Safety-2"
         (path "/1925ab50-b129-485f-aa70-9d722d7d68aa"
           (reference "#PWR04") (unit 1)
@@
     (pin "1")
     (instances
-      (project "Bike Safety"
+      (project "Bike Safety-2"
         (path "/1925ab50-b129-485f-aa70-9d722d7d68aa"
           (reference "#PWR012") (unit 1)
@@
     (pin "3")
     (instances
-      (project "Bike Safety"
+      (project "Bike Safety-2"
         (path "/1925ab50-b129-485f-aa70-9d722d7d68aa"
           (reference "U3") (unit 1)
@@
     (pin "4")
     (instances
-      (project "Bike Safety"
+      (project "Bike Safety-2"
         (path "/1925ab50-b129-485f-aa70-9d722d7d68aa"
           (reference "U2") (unit 1)
+        )
+      )
+    )
+  )
+  (symbol (lib_id "Device:R") (at 160.02 138.43 0) (unit 1)
+    (in_bom yes) (on_board yes) (dnp no)
+    (property "Reference" "R7" (at 154.94 138.43 90)
+      (effects (font (size 1.27 1.27)))
+    )
+    (property "Value" "10k" (at 157.48 138.43 90)
+      (effects (font (size 1.27 1.27)))
+    )
+    (property "Footprint" "" (at 158.242 138.43 90)
+      (effects (font (size 1.27 1.27)) hide)
+    )
+    (property "Datasheet" "~" (at 160.02 138.43 0)
+      (effects (font (size 1.27 1.27)) hide)
+    )
+    (pin "1")
+    (pin "2")
+    (instances
+      (project "Bike Safety-2"
+        (path "/1925ab50-b129-485f-aa70-9d722d7d68aa"
+          (reference "R7") (unit 1)
         )
       )
@@
     (pin "2")
     (instances
-      (project "Bike Safety"
+      (project "Bike Safety-2"
         (path "/1925ab50-b129-485f-aa70-9d722d7d68aa"
           (reference "BZ1") (unit 1)
@@
     (pin "1")
     (instances
-      (project "Bike Safety"
+      (project "Bike Safety-2"
         (path "/1925ab50-b129-485f-aa70-9d722d7d68aa"
           (reference "#PWR011") (unit 1)
@@
     (pin "1")
     (instances
-      (project "Bike Safety"
+      (project "Bike Safety-2"
         (path "/1925ab50-b129-485f-aa70-9d722d7d68aa"
           (reference "#PWR06") (unit 1)
@@
     (pin "1")
     (instances
-      (project "Bike Safety"
+      (project "Bike Safety-2"
         (path "/1925ab50-b129-485f-aa70-9d722d7d68aa"
           (reference "#PWR09") (unit 1)
@@
     (pin "2")
     (instances
-      (project "Bike Safety"
+      (project "Bike Safety-2"
         (path "/1925ab50-b129-485f-aa70-9d722d7d68aa"
           (reference "R2") (unit 1)
@@
     (pin "2")
     (instances
-      (project "Bike Safety"
+      (project "Bike Safety-2"
         (path "/1925ab50-b129-485f-aa70-9d722d7d68aa"
           (reference "D4") (unit 1)
         )
       )
+    )
+  )
+  (symbol (lib_id "Switch:SW_Push") (at 160.02 128.27 90) (unit 1)
+    (in_bom yes) (on_board yes) (dnp no) (fields_autoplaced)
+    (property "Reference" "SW1" (at 161.29 127 90)
+      (effects (font (size 1.27 1.27)) (justify right))
+    )
+    (property "Value" "SW_Push" (at 161.29 129.54 90)
+      (effects (font (size 1.27 1.27)) (justify right))
+    )
+    (property "Footprint" "" (at 154.94 128.27 0)
+      (effects (font (size 1.27 1.27)) hide)
+    )
+    (property "Datasheet" "~" (at 154.94 128.27 0)
+      (effects (font (size 1.27 1.27)) hide)
+    )
+    (pin "1")
+    (pin "2")
+    (instances
+      (project "Bike Safety-2"
+        (path "/1925ab50-b129-485f-aa70-9d722d7d68aa"
+          (reference "SW1") (unit 1)
+        )
+      )
